File: Hardware/ESP8266-Thing-Dev.brd (EAGLE design)
At the start: 55.2 x 25.7 mm, 69 parts, among them J1 DNP, Q1 MMBT2222A, Q2 MMBT2222A, U1 AP2112K-3.3V, U2 ESP8266, U3 AT25SF041-SOIC8, U4 FTS31XS-U, Y1 26MHz

Commit message: Schematic cleanup, tweaking silkscreen
Parts:
- removed SJ5: U.FL, SparkFun-Passives:PAD-JUMPER-2-NO_NO_SILK
- added SJ3: TRACE, SparkFun-Passives:PAD-JUMPER-2-NC_BY_PASTE_NO_SILK
- JP5: device SparkFun-Connectors:1X02 -> SparkFun-Connectors:1X02_NO_SILK
- SJ4: value TRACE -> U.FL; device SparkFun-Passives:PAD-JUMPER-2-NC_BY_PASTE_NO_SILK -> SparkFun-Passives:PAD-JUMPER-2-NO_NO_SILK
- moved SJ4 1.05 mm to (46.0, 13.9), turned to 90 degrees
- moved LOGO3 0.25 mm to (49.3, 1.65)
Connections:
- net ANT: now also SJ4.1; no longer SJ5.1
- net LNA2: now also SJ3.1, SJ4.2; no longer SJ4.1, SJ5.2
- net TRACE_ANT: now also SJ3.2; no longer SJ4.2
Routing:
- net N$14: track 9.63 -> 8.95 mm
Other:
- board text added: "!RST!"
- board text added: "4.5-6V"
